Commit message: Fix robot simulation errors

File: go2_description/xacro/robot.xacro (robot description, xacro)
@@ -6,13 +6,12 @@
     <xacro:include filename="$(find go2_description)/xacro/gz.xacro"/>
     <!-- Base Link -->
-    <link name="base_link">
-        <visual>
-            <origin rpy="0 0 0" xyz="0 0 0"/>
-            <geometry>
-                <box size="0.001 0.001 0.001"/>
-            </geometry>
-        </visual>
-    </link>
-    <joint name="floating_base" type="fixed">
+    <link name="base_footprint"/>
+    <link name="base_link"/>
+    <joint name="base_footprint_joint" type="fixed">
+        <origin rpy="0 0 0" xyz="0 0 0.32"/>
+        <parent link="base_footprint"/>
+        <child link="base_link"/>
+    </joint>
+    <joint name="trunk_joint" type="fixed">
         <origin rpy="0 0 0" xyz="0 0 0"/>
         <parent link="base_link"/>
@@ -54,57 +53,16 @@
     </joint>
     <!-- 2D Lidar -->
-    <link name="two_d_lidar">
-        <collision>
-            <origin xyz="0 0 0" rpy="0 0 0" />
-            <geometry>
-                <cylinder length="0.06" radius="0.075"/>
-            </geometry>
-        </collision>
-        <visual>
-            <origin xyz="0 0 0" rpy="0 0 0" />
-            <geometry>
-                <cylinder length="0.06" radius="0.075"/>
-            </geometry>
-        </visual>
-        <inertial>
-            <origin xyz="0 0 0" rpy="0 0 0" />
-            <mass value="0.1"/>
-            <xacro:cylinder_inertia m="0.1" r="0.075" h="0.06"/>
-        </inertial>
-    </link>
+    <link name="two_d_lidar"/>
     <joint name="two_d_lidar_joint" type="fixed">
         <parent link="base_link"/>
         <child link="two_d_lidar"/>
-        <origin xyz="0.2 0 0.08" rpy="0 0 0" />
+        <origin xyz="0.28945 0 -0.046825" rpy="0 2.8782 0" />
     </joint>
     <!-- Camera -->
-    <link name="kinect_camera">
-        <collision>
-            <origin xyz="0 0 0" rpy="0 0 0" />
-            <geometry>
-                <box size="0.07 0.3 0.09"/>
-            </geometry>
-        </collision>
-        <visual>
-            <origin xyz="0 0 0" rpy="0 0 0" />
-            <geometry>
-                <mesh filename="file://$(find go2_description)/meshes/kinect/d415.dae"/>
-            </geometry>
-        </visual>
-        <inertial>
-            <mass value="0.01"/>
-            <xacro:box_inertia m="0.01" x="0.07" y="0.3" z = "0.09"/>
-        </inertial>
-    </link>
+    <link name="kinect_camera"/>
     <joint name="kinect_camera_joint" type="fixed">
-        <origin rpy="0 0 0" xyz="${trunk_length/2} 0 ${trunk_height/7}"/>
+        <origin rpy="0 0 0" xyz="0.32715 -0.00003 0.04297"/>
         <parent link="base_link"/>
         <child link="kinect_camera"/>
     </joint>
-    <link name="kinect_camera_optical"/>
-    <joint name="kinect_camera_optical_joint" type="fixed">
-        <origin xyz="0 0 0" rpy="${-pi/2} 0 ${-pi/2}"/>
-        <parent link="kinect_camera"/>
-        <child link="kinect_camera_optical"/>
-    </joint>
 </robot>
