Commit message: Add champ controller

File: go2_description/xacro/gz.xacro (robot description, xacro)
@@ -1,4 +1,11 @@
 <?xml version="1.0"?>
 <robot xmlns:xacro="http://www.ros.org/wiki/xacro">
+    <!-- ROS2 Control -->
+    <gazebo>
+        <plugin filename="gz_ros2_control-system" name="gz_ros2_control::GazeboSimROS2ControlPlugin">
+            <parameters>$(find go2_description)/config/ros_control.yaml</parameters>
+            <ros><remapping>/controller_manager/robot_description:=/robot_description</remapping></ros>
+        </plugin>
+    </gazebo>
     <!-- ........................... SENSOR PLUGIN ................................... -->
     <gazebo>

File: go2_description/xacro/leg.xacro (robot description, xacro)
@@ -150,4 +150,24 @@
             </inertial>
         </link>
+        <ros2_control name="${name}" type="system">
+            <hardware>
+                <plugin>gz_ros2_control/GazeboSimSystem</plugin>
+            </hardware>
+            <joint name="${name}_hip_joint">
+                <command_interface name="effort"/>
+                <state_interface name="position"/>
+                <state_interface name="velocity"/>
+            </joint>
+            <joint name="${name}_upper_leg_joint">
+                <command_interface name="effort"/>
+                <state_interface name="position"/>
+                <state_interface name="velocity"/>
+            </joint>
+            <joint name="${name}_lower_leg_joint">
+                <command_interface name="effort"/>
+                <state_interface name="position"/>
+                <state_interface name="velocity"/>
+            </joint>
+        </ros2_control>
     </xacro:macro>
 </robot>

File: go2_description/xacro/robot.xacro (robot description, xacro)
@@ -6,12 +6,6 @@
     <xacro:include filename="$(find go2_description)/xacro/gz.xacro"/>
     <!-- Base Link -->
-    <link name="base_footprint"/>
     <link name="base_link"/>
-    <joint name="base_footprint_joint" type="fixed">
-        <origin rpy="0 0 0" xyz="0 0 0.32"/>
-        <parent link="base_footprint"/>
-        <child link="base_link"/>
-    </joint>
-    <joint name="trunk_joint" type="fixed">
+    <joint name="floating_base" type="fixed">
         <origin rpy="0 0 0" xyz="0 0 0"/>
         <parent link="base_link"/>
