Commit message: Complete go2_description package

File: go2_description/xacro/const.xacro (robot description, xacro)
@@ -100,35 +100,3 @@
     <!-- foot -->
     <xacro:property name="foot_mass" value="0.06"/>
-    <!-- sensors -->
-    <xacro:property name="two_d_lidar_update_rate" value="30"/>
-    <xacro:property name="two_d_lidar_sample_size" value="361"/>
-    <xacro:property name="two_d_lidar_min_angle" value="0"/>
-    <xacro:property name="two_d_lidar_max_angle" value="360"/>
-    <xacro:property name="two_d_lidar_min_range" value="0.55"/>
-    <xacro:property name="two_d_lidar_max_range" value="16"/>
-    <xacro:property name="camera_baseline" value="0.06"/>
-    <xacro:property name="camera_height" value="0.10"/>
-    <xacro:property name="camera_horizontal_fov" value="60"/>
-    <xacro:arg name="robot_namespace" default=""/>
-    <xacro:arg name="wheel_odom_topic" default="odom" />
-    <xacro:arg name="camera_enabled" default="false" />
-    <xacro:arg name="stereo_camera_enabled" default="false" />
-    <xacro:arg name="two_d_lidar_enabled" default="false" />
-    <xacro:arg name="publish_wheel_odom_tf" default="true" />
-    <xacro:arg name="conveyor_enabled" default="false"/>
-    <xacro:arg name="ground_truth_frame" default="map"/>
-    <xacro:arg name="sim_gazebo" default="false" />
-    <xacro:arg name="sim_ign" default="false" />
-    <xacro:arg name="sim_gz" default="false" />
-    <xacro:arg name="odometry_source" default="world" />
-    <!--................................ INERTIA MATRICES .............................. -->
-    <xacro:macro name="cylinder_inertia" params="m r h">
-        <inertia ixx="${m * (3 * r * r + h * h) / 12}" ixy="0" ixz="0" iyy="${m * (3 * r * r + h * h) / 12}" iyz="0" izz="${m * r * r / 2}" />
-    </xacro:macro>
-    <xacro:macro name="box_inertia" params="m x y z">
-        <inertia ixx="${m * (y * y + z * z) / 12}" ixy="0" ixz="0" iyy="${m * (x * x + z * z) / 12}" iyz="0" izz="${m * (y * y + x * x) / 12}" />
-    </xacro:macro>
-    <xacro:macro name="sphere_inertia" params="m r">
-        <inertia ixx="${2 * m * r * r / 5}" ixy="0" ixz="0" iyy="${2 * m * r * r / 5}" iyz="0" izz="${2 * m * r * r / 5}" />
-    </xacro:macro>
 </robot>

File: go2_description/xacro/gz.xacro (robot description, xacro)
@@ -8,44 +8,42 @@
         </plugin>
     </gazebo>
-    <!-- ........................... SENSOR PLUGIN ................................... -->
+    <!-- Sensor Plugins -->
     <gazebo>
         <plugin filename="gz-sim-sensors-system" name="gz::sim::systems::Sensors">
             <render_engine>ogre2</render_engine>
         </plugin>
-        <plugin filename="gz-sim-imu-system" name="gz::sim::systems::Imu">
-        </plugin>
-        <plugin filename="gz-sim-joint-state-publisher-system" name="gz::sim::systems::JointStatePublisher">
-        </plugin>
+        <plugin filename="gz-sim-imu-system" name="gz::sim::systems::Imu"/>
+        <plugin filename="gz-sim-joint-state-publisher-system" name="gz::sim::systems::JointStatePublisher"/>
     </gazebo>
-    <!-- ............................. ground truth .................................... -->
+    <!-- Odometry -->
     <gazebo>
         <plugin filename="libgz-sim-odometry-publisher-system"
             name="gz::sim::systems::OdometryPublisher">
             <odom_frame>odom</odom_frame>
-            <robot_base_frame>base_footprint</robot_base_frame>
-            <odom_topic>$(arg wheel_odom_topic)</odom_topic>
-            <tf_topic>/tf</tf_topic>
+            <robot_base_frame>base_link</robot_base_frame>
+            <odom_topic>odom</odom_topic>
+            <tf_topic>tf</tf_topic>
             <dimensions>2</dimensions>
             <odom_publish_frequency>10</odom_publish_frequency>
         </plugin>
     </gazebo>
-    <!-- ........................... 2D LIDAR config ................................... -->
-    <gazebo reference="two_d_lidar">
-        <sensor name='gpu_lidar' type='gpu_lidar'>
+    <!-- Lidar -->
+    <gazebo reference="lidar_link">
+        <sensor name="gpu_lidar" type="gpu_lidar">
             <topic>scan</topic>
-            <update_rate>${two_d_lidar_update_rate}</update_rate>
-            <gz_frame_id>two_d_lidar</gz_frame_id>
+            <update_rate>50</update_rate>
+            <gz_frame_id>lidar_link</gz_frame_id>
             <lidar>
                 <scan>
                     <horizontal>
-                        <samples>${two_d_lidar_sample_size}</samples>
+                        <samples>440</samples>
                         <resolution>1</resolution>
-                        <min_angle>${radians(two_d_lidar_min_angle)}</min_angle>
-                        <max_angle>${radians(two_d_lidar_max_angle)}</max_angle>
+                        <min_angle>-3.141592653589793</min_angle>
+                        <max_angle>3.141592653589793</max_angle>
                     </horizontal>
                 </scan>
                 <range>
-                    <min>${two_d_lidar_min_range}</min>
-                    <max>${two_d_lidar_max_range}</max>
+                    <min>0.3</min>
+                    <max>3.5</max>
                     <resolution>0.01</resolution>
                 </range>
@@ -53,5 +51,5 @@
                     <type>gaussian</type>
                     <mean>0.0</mean>
-                    <stddev>0.001</stddev>
+                    <stddev>0.01</stddev>
                 </noise>
             </lidar>
@@ -60,13 +58,12 @@
         </sensor>
     </gazebo>
-    <!-- ........................... CAMERA config ................................... -->
-    <gazebo reference="kinect_camera">
-        <sensor type="depth_camera" name="kinect_camera">
+    <!-- Camera -->
+    <gazebo reference="camera_link">
+        <sensor type="camera" name="camera">
             <update_rate>30.0</update_rate>
-            <topic>kinect_camera</topic>
-            <gz_frame_id>kinect_camera</gz_frame_id>
+            <topic>camera</topic>
+            <gz_frame_id>camera_link</gz_frame_id>
             <camera>
-                <camera_info_topic>kinect_camera/camera_info</camera_info_topic>
-                <horizontal_fov>${radians(camera_horizontal_fov)}</horizontal_fov>
+                <camera_info_topic>camera/camera_info</camera_info_topic>
                 <image>
                     <width>640</width>
@@ -74,21 +71,18 @@
                     <format>R8G8B8</format>
                 </image>
-                <clip>
-                    <near>0.05</near>
-                    <far>8.0</far>
-                </clip>
             </camera>
         </sensor>
     </gazebo>
-    <!-- ........................... IMU config ................................... -->
-    <gazebo reference="imu_frame">
+    <!-- IMU -->
+    <gazebo reference="imu_link">
         <sensor name="imu_sensor" type="imu">
             <always_on>1</always_on>
-            <update_rate>1</update_rate>
-            <gz_frame_id>imu_frame</gz_frame_id>
+            <update_rate>50</update_rate>
+            <frame_id>imu_frame</frame_id>
             <visualize>true</visualize>
-            <topic>imu</topic>
+            <topic>imu/data</topic>
         </sensor>
     </gazebo>
+    <!-- Physical Parameters -->
     <gazebo reference="trunk">
         <mu1>0.2</mu1>
@@ -97,12 +91,4 @@
         <kd>0.5</kd>
     </gazebo>
-    <!-- <gazebo reference="stick_link">
-        <mu1>0.2</mu1>
-        <mu2>0.2</mu2>
-    </gazebo> -->
-    <!-- <gazebo reference="imu_link">
-        <mu1>0.2</mu1>
-        <mu2>0.2</mu2>
-    </gazebo> -->
     <!-- FL leg -->
     <gazebo reference="lf_hip_link">

File: go2_description/xacro/leg.xacro (robot description, xacro)
@@ -124,5 +124,5 @@
             </inertial>
         </link>
-        <joint name="${name}_foot_joint" type="fixed">0
+        <joint name="${name}_foot_joint" type="fixed">
             <origin rpy="0 0 0" xyz="0 0 ${-(calf_length)}"/>
             <parent link="${name}_lower_leg_link"/>

File: go2_description/xacro/robot.xacro (robot description, xacro)
@@ -40,23 +40,23 @@
     <xacro:leg name="lh" mirror="1"  mirror_dae="True"   front_hind="-1" front_hind_dae="False"/>
     <!-- IMU -->
-    <link name="imu_frame"/>
+    <link name="imu_link"/>
     <joint name="imu_joint" type="fixed">
         <parent link="trunk"/>
-        <child link="imu_frame"/>
+        <child link="imu_link"/>
         <origin rpy="0 0 0" xyz="0 0 0"/>
     </joint>
-    <!-- 2D Lidar -->
-    <link name="two_d_lidar"/>
-    <joint name="two_d_lidar_joint" type="fixed">
+    <!-- Lidar -->
+    <link name="lidar_link"/>
+    <joint name="lidar_joint" type="fixed">
         <parent link="base_link"/>
-        <child link="two_d_lidar"/>
-        <origin xyz="0.28945 0 -0.046825" rpy="0 2.8782 0" />
+        <child link="lidar_link"/>
+        <origin xyz="0.225 0 0.105" rpy="0 0 0" />
     </joint>
     <!-- Camera -->
-    <link name="kinect_camera"/>
-    <joint name="kinect_camera_joint" type="fixed">
+    <link name="camera_link"/>
+    <joint name="camera_joint" type="fixed">
         <origin rpy="0 0 0" xyz="0.32715 -0.00003 0.04297"/>
         <parent link="base_link"/>
-        <child link="kinect_camera"/>
+        <child link="camera_link"/>
     </joint>
 </robot>
